File: keeb/main.kicad_pcb (KiCad board)
At the start: 2 copper layers, 115 x 78 mm, 38 parts

Commit message: First PCB
Parts:
- removed the ? at (25.0, 15.0)
- added REF**: VIA-0.6mm, VIA-0.6mm, F.Cu at (108.0, -47.0)
- added REF**: VIA-0.6mm, VIA-0.6mm, F.Cu at (110.0, -47.0)
- moved ? 59.3 mm to (108.0, -51.5), turned to 180 degrees
- moved ? 23.9 mm to (110.0, -18.0), turned to 270 degrees
- moved S33 13.2 mm to (105.0, 21.6), turned to 45 degrees
- moved S34 13.2 mm to (105.0, 21.6), turned to 225 degrees
- moved MCU1 7.81 mm to (110.0, -35.0)
- moved S31 5.83 mm to (85.0, 10.0)
- moved S32 5.83 mm to (85.0, 10.0)
- moved S10 5.00 mm to (36.0, -27.0)
- moved S11 5.00 mm to (36.0, -44.0)
- moved S12 5.00 mm to (36.0, -44.0)
- moved S19 5.00 mm to (72.0, -10.0)
- moved S20 5.00 mm to (72.0, -10.0)
- moved S21 5.00 mm to (72.0, -27.0)
- moved S22 5.00 mm to (72.0, -27.0)
- moved S23 5.00 mm to (72.0, -44.0)
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Connections:
- S1 pad 1: P21 -> P3
- S10 pad 1: P15 -> P0
- S11 pad 1: P14 -> P18
- S12 pad 1: P14 -> P18
- S13 pad 1: P16 -> P5
- S14 pad 1: P16 -> P5
- S15 pad 1: P10 -> P14
- S16 pad 1: P10 -> P14
- S17 pad 1: P4 -> P19
- S18 pad 1: P4 -> P19
- S19 pad 1: P5 -> P6
- S2 pad 1: P21 -> P3
- S20 pad 1: P5 -> P6
- S21 pad 1: P6 -> P10
- S22 pad 1: P6 -> P10
- S23 pad 1: P9 -> P20
- S24 pad 1: P9 -> P20
- S27 pad 1: P8 -> P16
- S28 pad 1: P8 -> P16
- S29 pad 1: P3 -> P21
- S3 pad 1: P20 -> P2
- S30 pad 1: P3 -> P21
- S31 pad 1: P2 -> P8
- S32 pad 1: P2 -> P8
- S33 pad 1: P1 -> P9
- S34 pad 1: P1 -> P9
- S4 pad 1: P20 -> P2
- S5 pad 1: P19 -> P15
- S6 pad 1: P19 -> P15
- S7 pad 1: P18 -> P4
- S8 pad 1: P18 -> P4
- S9 pad 1: P15 -> P0
Other:
- board size 115 x 78 mm -> 113.1 x 94.6 mm
